File: hardware/xen_teensy_motherboard_matrix_mki.sch (EAGLE design)
At the start: 221 parts, among them IC1 TL074PW, IC10 MCP4351-104E_ST, IC11 MCP4351-104E_ST, IC12 MCP4351-104E_ST, IC13 MCP4351-104E_ST, IC14 MCP4351-104E_ST, IC15 MCP4351-104E_ST, IC16 MCP4351-104E_ST, IC17 MCP4351-104E_ST, IC2 TL074PW, IC3 MCP6004, IC4 MCP4351-104E_ST, IC5 TL074PW, IC6 TEENSY41-OUTER, IC7 R-78E5.0-0.5, IC8 LM4040-5V, IC9 LD2981 3.3V

Commit message: add offset to input and output voltages
Parts:
- added R78, R79, R80, R81, R82, R83, R84, R85, R86, R87, R88, R89: 100k, resistors:RESISTOR
- R1, R16, R20, R39, R4, R42, R46, R74, R75, R76, R77, R9: value 100k -> 200k
- R10, R17, R19, R2, R21, R22, R23, R24, R25, R26, R27, R28, R30, R31, R32, R33, R34, R35, R36, R37, R38, R40, R43, R45, R47, R48, R49, R5, R50, R51, R52, R53, R54, R55, R56, R57, R58, R59, R60, R61, R72, R73: value 100k -> 47k
Connections:
- net -5VREF: now also R78.1, R79.1, R80.1, R81.1, R82.1, R83.1, R84.1, R85.1, R86.1, R87.1, R88.1, R89.1
- net N$12: now also R80.2
- net N$2: now also R82.2
- net N$20: now also R81.2
- net N$28: now also R78.2
- net N$48: now also R83.2
- net N$50: now also R79.2
- net OUT1: now also R85.2
- net OUT2: now also R89.2
- net OUT3: now also R87.2
- net OUT4: now also R88.2
- net OUT5: now also R86.2
- net OUT6: now also R84.2

Commit message: buffer calibration voltage
Parts:
- added IC18: TL072W, ic_analogue:TL072W
- added R93: 100k, resistors:TRIMMER64X
- added R94, R95: 47k, resistors:RESISTOR
- R84, R85, R87: value 100k -> 16.6k
Connections:
- removed net N$74: IC6.3V3-1
- new net N$21: IC18B.-IN, IC18B.OUT
- new net N$43: R93.E, R95.2
- new net N$49: R93.A, R94.1
- new net N$5: IC10.P0B, IC10.P1B, IC10.P2B, IC10.P3B, IC11.P0B, IC11.P1B, IC11.P2B, IC11.P3B, IC12.P0B, IC12.P1B, IC12.P2B, IC12.P3B, IC13.P0B, IC13.P1B, IC13.P2B, IC13.P3B, IC14.P0B, IC14.P1B, IC14.P2B, IC14.P3B, IC15.P0B, IC15.P1B, IC15.P2B, IC15.P3B, IC16.P0B, IC16.P1B, IC16.P2B, IC16.P3B, IC17.P0B, IC17.P1B, IC17.P2B, IC17.P3B, IC18A.-IN, IC18A.OUT, IC4.P0B, IC4.P1B, IC4.P2B, IC4.P3B
- new net N$9: IC18A.+IN, R93.S
- new net SDO: IC10.SDO, IC11.SDO, IC12.SDO, IC13.SDO, IC14.SDO, IC15.SDO, IC16.SDO, IC17.SDO, IC4.SDO
- net +12V: now also IC18P.V+
- net -12V: now also IC18P.V-
- net 3.3V: no longer IC10.VDD, IC11.VDD, IC12.VDD, IC13.VDD, IC14.VDD, IC15.VDD, IC16.VDD, IC17.VDD, IC4.VDD
- net 5V: now also IC10.VDD, IC11.VDD, IC12.VDD, IC13.VDD, IC14.VDD, IC15.VDD, IC16.VDD, IC17.VDD, IC4.VDD, R94.2
- net PE: now also IC18B.+IN, R95.1; no longer IC10.P0B, IC10.P1B, IC10.P2B, IC10.P3B, IC11.P0B, IC11.P1B, IC11.P2B, IC11.P3B, IC12.P0B, IC12.P1B, IC12.P2B, IC12.P3B, IC13.P0B, IC13.P1B, IC13.P2B, IC13.P3B, IC14.P0B, IC14.P1B, IC14.P2B, IC14.P3B, IC15.P0B, IC15.P1B, IC15.P2B, IC15.P3B, IC16.P0B, IC16.P1B, IC16.P2B, IC16.P3B, IC17.P0B, IC17.P1B, IC17.P2B, IC17.P3B, IC4.P0B, IC4.P1B, IC4.P2B, IC4.P3B
- net SPI_MISO: no longer IC10.SDO, IC11.SDO, IC12.SDO, IC13.SDO, IC14.SDO, IC15.SDO, IC16.SDO, IC17.SDO, IC4.SDO
Other:
- note added: "ADJUST TO 2.35V"
